File: target_node/board/v1.sch (EAGLE design)
At the start: 13 parts, among them IC1 UA741P, U1 L78XXAB/AC/V

Commit message: Changed schematic to connect nRF24 board to other digital outputs and make a single layer board
Parts:
- removed POWER: 22-23-2021, con-molex:22-23-2021
Connections:
- removed net GND: C2.1, IC1.V-, NRF24L01.2, PIEZO-1.S, POWER-2.S, R1.1, RGB_LED.2, U$2.GND, U1.IN
- removed net N$4: NRF24L01.4, U$2.7
- new net N$15: NRF24L01.3, U$2.A1
- new net N$17: NRF24L01.2, U$2.GND@2, U1.IN
- new net N$18: C2.1, IC1.V-, PIEZO-1.S, R1.1, RGB_LED.2, U$2.GND
- net N$5: now also NRF24L01.4, U$2.A0; no longer NRF24L01.3, U$2.8
- net VCC: no longer POWER-1.S
Other:
- moved on the sheet: R1
